File: HW/TI-LAB/TI-LAB.sch (KiCad schematic (older format))
At the start: 113 parts, among them J1 V+, J2 GND, J4 PWR, U1 OpAmp, U10 OpAmp, U2 OpAmp, U3 OpAmp, U4 OpAmp, U5 OpAmp, U6 OpAmp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

Commit message: add reimaing - archive
Parts:
- gave numbers to parts that had none: 3
- renumbered C2 to C3
Connections:
- net Output2: now also TP5.1, TP5.2, Vout2.1 (In)
